File: boards/shuchir_jain_snoweo/light_controller.kicad_pcb (KiCad board)
At the start: 2 copper layers, 65.2 x 57.5 mm, 28 parts, among them J1 RJ45, J2 Conn_02x05_Odd_Even, J3 2157601003, J4 2157601003, SW1 SW_Push, U1 STM32F103C8Tx, U2 ISO1050DUB, U3 AMS1117-3.3, U4 SN74LV1T34DBV, U5 SN74LV1T34DBV

Commit message: move imported components to local libs
Parts:
- J3, J4: footprint SamacSys:215760YY03 -> samacsys-evc:215760YY03
