File: boards/shuchir_jain_snoweo/light_controller.kicad_sch (KiCad schematic)
At the start: 28 parts, among them J1 RJ45, J2 Conn_02x05_Odd_Even, J3 2157601003, J4 2157601003, SW1 SW_Push, U1 STM32F103C8Tx, U2 ISO1050DUB, U3 AMS1117-3.3, U4 SN74LV1T34DBV, U5 SN74LV1T34DBV

Commit message: move imported components to local libs
Parts:
- J3, J4: footprint SamacSys:215760YY03 -> samacsys-evc:215760YY03; symbol SamacSys:2157601003 -> samacsys-evc:2157601003
Changed lines of the file:
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@@
 	)
 	(symbol
-		(lib_id "SamacSys:2157601003")
+		(lib_id "samacsys-evc:2157601003")
 		(at 83.82 29.21 0)
 		(unit 1)
@@
 			)
 		)
-		(property "Footprint" "SamacSys:215760YY03"
+		(property "Footprint" "samacsys-evc:215760YY03"
 			(at 100.33 124.13 0)
 			(hide yes)
@@
 	)
 	(symbol
-		(lib_id "SamacSys:2157601003")
+		(lib_id "samacsys-evc:2157601003")
 		(at 83.82 53.34 0)
 		(unit 1)
@@
 			)
 		)
-		(property "Footprint" "SamacSys:215760YY03"
+		(property "Footprint" "samacsys-evc:215760YY03"
 			(at 100.33 148.26 0)
 			(hide yes)
